File: medidor/medidor.sch (KiCad schematic (older format))
At the start: 17 parts, among them J1 Screw_Terminal_01x02, J2 Conn_01x01_Female, J3 Conn_01x01_Female, U1 LTC1966CMS8PBF, U2 MCP6001U

Commit message: Se asocian los footprints
Parts:
- C1: footprint (none) -> Capacitor_SMD:C_1206_3216Metric_Pad1.42x1.75mm_HandSolder
- C2, C4: footprint (none) -> Capacitor_SMD:CP_Elec_6.3x4.9
- C3, C5: footprint (none) -> Capacitor_SMD:C_0805_2012Metric_Pad1.15x1.40mm_HandSolder
- J1: footprint (none) -> TerminalBlock_MetzConnect:TerminalBlock_MetzConnect_Type703_RT10N02HGLU_1x02_P9.52mm_Horizontal
- J2, J3: footprint (none) -> Connector_PinHeader_2.54mm:PinHeader_1x01_P2.54mm_Vertical
- JP1, JP2: footprint (none) -> Jumper:SolderJumper-2_P1.3mm_Open_RoundedPad1.0x1.5mm
- R1: footprint (none) -> Resistor_THT:R_Axial_Power_L60.0mm_W14.0mm_P71.12mm
- R2, R3, R4: footprint (none) -> Resistor_SMD:R_0805_2012Metric_Pad1.15x1.40mm_HandSolder
- RV1: footprint (none) -> Potentiometer_SMD:Potentiometer_Bourns_TC33X_Vertical
- U1: footprint MSOP-8_MS -> LTC1966CMS8PBF:MSOP-8_MS
- U2: footprint (none) -> Package_TO_SOT_SMD:SOT-353_SC-70-5_Handsoldering
Changed lines of the file:
@@
 F 0 "U1" H 3850 1715 50  0000 C CNN
 F 1 "LTC1966CMS8PBF" H 3850 1624 50  0000 C CNN
-F 2 "MSOP-8_MS" H 2950 1350 50  0001 L BNN
+F 2 "LTC1966CMS8PBF:MSOP-8_MS" H 2950 1350 50  0001 L BNN
 F 3 "" H 2950 1350 50  0001 L BNN
 F 4 "Linear Technology" H 2950 1350 50  0001 L BNN "VENDOR"
@@
 F 0 "JP2" H 6450 1464 50  0000 C CNN
 F 1 "Jumper" H 6450 1373 50  0000 C CNN
-F 2 "" H 6450 1200 50  0001 C CNN
+F 2 "Jumper:SolderJumper-2_P1.3mm_Open_RoundedPad1.0x1.5mm" H 6450 1200 50  0001 C CNN
 F 3 "~" H 6450 1200 50  0001 C CNN
 	1    6450 1200
@@
 F 0 "J3" V 6738 862 50  0000 R CNN
 F 1 "Conn_01x01_Female" V 6647 862 50  0000 R CNN
-F 2 "" H 6800 950 50  0001 C CNN
+F 2 "Connector_PinHeader_2.54mm:PinHeader_1x01_P2.54mm_Vertical" H 6800 950 50  0001 C CNN
 F 3 "~" H 6800 950 50  0001 C CNN
 	1    6800 950
@@
 F 0 "C5" H 6215 1446 50  0000 L CNN
 F 1 "100nF" H 6215 1355 50  0000 L CNN
-F 2 "" H 6138 1250 50  0001 C CNN
+F 2 "Capacitor_SMD:C_0805_2012Metric_Pad1.15x1.40mm_HandSolder" H 6138 1250 50  0001 C CNN
 F 3 "~" H 6100 1400 50  0001 C CNN
 	1    6100 1400
@@
 F 0 "C4" H 5868 1446 50  0000 L CNN
 F 1 "1uF" H 5868 1355 50  0000 L CNN
-F 2 "" H 5788 1250 50  0001 C CNN
+F 2 "Capacitor_SMD:CP_Elec_6.3x4.9" H 5788 1250 50  0001 C CNN
 F 3 "~" H 5750 1400 50  0001 C CNN
 	1    5750 1400
@@
 F 0 "U2" H 2800 4750 50  0000 L CNN
 F 1 "MCP6001U" H 2650 4650 50  0000 L CNN
-F 2 "" H 2600 4500 50  0001 L CNN
+F 2 "Package_TO_SOT_SMD:SOT-353_SC-70-5_Handsoldering" H 2600 4500 50  0001 L CNN
 F 3 "http://ww1.microchip.com/downloads/en/DeviceDoc/21733j.pdf" H 2600 4500 50  0001 C CNN
 	1    2600 4500
@@
 F 0 "J1" H 1418 1375 50  0000 C CNN
 F 1 "Screw_Terminal_01x02" H 1750 1450 50  0000 C CNN
-F 2 "" H 1500 1700 50  0001 C CNN
+F 2 "TerminalBlock_MetzConnect:TerminalBlock_MetzConnect_Type703_RT10N02HGLU_1x02_P9.52mm_Horizontal" H 1500 1700 50  0001 C CNN
 F 3 "~" H 1500 1700 50  0001 C CNN
 	1    1500 1700
@@
 F 0 "R1" H 1920 1696 50  0000 L CNN
 F 1 "0.1" H 1920 1605 50  0000 L CNN
-F 2 "" V 1780 1650 50  0001 C CNN
+F 2 "Resistor_THT:R_Axial_Power_L60.0mm_W14.0mm_P71.12mm" V 1780 1650 50  0001 C CNN
 F 3 "~" H 1850 1650 50  0001 C CNN
 	1    1850 1650
@@
 F 0 "C1" V 1848 1450 50  0000 C CNN
 F 1 "3.9nF" V 1939 1450 50  0000 C CNN
-F 2 "" H 2138 1300 50  0001 C CNN
+F 2 "Capacitor_SMD:C_1206_3216Metric_Pad1.42x1.75mm_HandSolder" H 2138 1300 50  0001 C CNN
 F 3 "~" H 2100 1450 50  0001 C CNN
 	1    2100 1450
@@
 F 0 "R3" H 2270 5346 50  0000 L CNN
 F 1 "1k" H 2270 5255 50  0000 L CNN
-F 2 "" V 2130 5300 50  0001 C CNN
+F 2 "Resistor_SMD:R_0805_2012Metric_Pad1.15x1.40mm_HandSolder" V 2130 5300 50  0001 C CNN
 F 3 "~" H 2200 5300 50  0001 C CNN
 	1    2200 5300
@@
 F 0 "R4" H 2570 5096 50  0000 L CNN
 F 1 "6.8k" H 2570 5005 50  0000 L CNN
-F 2 "" V 2430 5050 50  0001 C CNN
+F 2 "Resistor_SMD:R_0805_2012Metric_Pad1.15x1.40mm_HandSolder" V 2430 5050 50  0001 C CNN
 F 3 "~" H 2500 5050 50  0001 C CNN
 	1    2500 5050
@@
 F 0 "R2" H 2120 4446 50  0000 L CNN
 F 1 "0" H 2120 4355 50  0000 L CNN
-F 2 "" V 1980 4400 50  0001 C CNN
+F 2 "Resistor_SMD:R_0805_2012Metric_Pad1.15x1.40mm_HandSolder" V 1980 4400 50  0001 C CNN
 F 3 "~" H 2050 4400 50  0001 C CNN
 	1    2050 4400
@@
 F 0 "RV1" H 2931 4896 50  0000 R CNN
 F 1 "R_POT" H 2931 4805 50  0000 R CNN
-F 2 "" H 3000 4850 50  0001 C CNN
+F 2 "Potentiometer_SMD:Potentiometer_Bourns_TC33X_Vertical" H 3000 4850 50  0001 C CNN
 F 3 "~" H 3000 4850 50  0001 C CNN
 	1    3000 4850
@@
 F 0 "JP1" H 3400 4764 50  0000 C CNN
 F 1 "Jumper" H 3400 4673 50  0000 C CNN
-F 2 "" H 3400 4500 50  0001 C CNN
+F 2 "Jumper:SolderJumper-2_P1.3mm_Open_RoundedPad1.0x1.5mm" H 3400 4500 50  0001 C CNN
 F 3 "~" H 3400 4500 50  0001 C CNN
 	1    3400 4500
@@
 F 0 "J2" V 3688 4162 50  0000 R CNN
 F 1 "Conn_01x01_Female" V 3597 4162 50  0000 R CNN
-F 2 "" H 3750 4250 50  0001 C CNN
+F 2 "Connector_PinHeader_2.54mm:PinHeader_1x01_P2.54mm_Vertical" H 3750 4250 50  0001 C CNN
 F 3 "~" H 3750 4250 50  0001 C CNN
 	1    3750 4250
@@
 F 0 "C2" H 4818 2396 50  0000 L CNN
 F 1 "10uF" H 4818 2305 50  0000 L CNN
-F 2 "" H 4738 2200 50  0001 C CNN
+F 2 "Capacitor_SMD:CP_Elec_6.3x4.9" H 4738 2200 50  0001 C CNN
 F 3 "~" H 4700 2350 50  0001 C CNN
 	1    4700 2350
@@
 F 0 "C3" H 5165 2396 50  0000 L CNN
 F 1 "100nF" H 5165 2305 50  0000 L CNN
-F 2 "" H 5088 2200 50  0001 C CNN
+F 2 "Capacitor_SMD:C_0805_2012Metric_Pad1.15x1.40mm_HandSolder" H 5088 2200 50  0001 C CNN
 F 3 "~" H 5050 2350 50  0001 C CNN
 	1    5050 2350

Commit message: Se agrega ruteo pcb y recuadros para cada parte dell esquematico
Parts:
- added J4: Conn_01x06, Connector_PinHeader_2.54mm:PinHeader_1x06_P2.54mm_Vertical, symbol Connector_Generic:Conn_01x06
- added J5: Screw_Terminal_01x02, TerminalBlock_MetzConnect:TerminalBlock_MetzConnect_Type703_RT10N02HGLU_1x02_P9.52mm_Horizontal, symbol Connector:Screw_Terminal_01x02
- added JP3: Fase_1, Jumper:SolderJumper-2_P1.3mm_Open_RoundedPad1.0x1.5mm, symbol Device:Jumper
- added JP4: Fase_2, Jumper:SolderJumper-2_P1.3mm_Open_RoundedPad1.0x1.5mm, symbol Device:Jumper
- added JP5: Fase_3, Jumper:SolderJumper-2_P1.3mm_Open_RoundedPad1.0x1.5mm, symbol Device:Jumper
- added JP6: Neutral, Jumper:SolderJumper-2_P1.3mm_Open_RoundedPad1.0x1.5mm, symbol Device:Jumper
Connections:
- net GND: now also J4.5 (Pin_5), J5.1 (Pin_1)
- net VDD: now also J4.6 (Pin_6)
- net CT_INPUT_2: now reaches C1.2, J1.2 (Pin_2), R1.1
- net CT_INPUT_2: now also J5.2 (Pin_2)
- net OUT_MCP6001u: now reaches J2.1 (Pin_1), JP1.2
- net OUT_MCP6001u: now also JP3.1, JP4.1, JP5.1, JP6.1
- new net Fase_1: J4.1 (Pin_1), JP3.2
- new net Fase_2: J4.2 (Pin_2), JP4.2
- new net Fase_3: J4.3 (Pin_3), JP5.2
- new net Neutral: J4.4 (Pin_4), JP6.2
Other:
- note added: "CURRENT TRANSFORMER INPUT"
- moved on the sheet: C1, C2, C3, C4, C5, J1, J3, JP2, R1, U1

Commit message: Se agrega PWR_FLAG para solucionar error de ERC
Changed lines of the file:
@@
 $EndComp
 Wire Wire Line
-	8200 4850 8300 4850
+	8200 4850 8250 4850
 Text Label 3800 4500 0    50   ~ 0
 OUT_MCP6001u
@@
 Wire Wire Line
 	2100 1850 2050 1850
+$Comp
+L power:PWR_FLAG #FLG0101
+U 1 1 607BC614
+P 8250 5050
+F 0 "#FLG0101" H 8250 5125 50  0001 C CNN
+F 1 "PWR_FLAG" H 8250 5229 50  0000 C CNN
+F 2 "" H 8250 5050 50  0001 C CNN
+F 3 "~" H 8250 5050 50  0001 C CNN
+	1    8250 5050
+	-1   0    0    1
+$EndComp
+Wire Wire Line
+	8250 5050 8250 4850
+Connection ~ 8250 4850
+Wire Wire Line
+	8250 4850 8300 4850
 $EndSCHEMATC

Commit message: Se agregan fiduciarios
Parts:
- added FID1, FID2, FID3: Fiducial, Fiducial:Fiducial_1.5mm_Mask4.5mm, symbol Mechanical:Fiducial
Changed lines of the file:
@@
 Wire Wire Line
 	8250 4850 8300 4850
+$Comp
+L Mechanical:Fiducial FID1
+U 1 1 607C8551
+P 10100 4300
+F 0 "FID1" H 10185 4347 50  0000 L CNN
+F 1 "Fiducial" H 10185 4254 50  0000 L CNN
+F 2 "Fiducial:Fiducial_1.5mm_Mask4.5mm" H 10100 4300 50  0001 C CNN
+F 3 "~" H 10100 4300 50  0001 C CNN
+	1    10100 4300
+	1    0    0    -1
+$EndComp
+$Comp
+L Mechanical:Fiducial FID2
+U 1 1 607C893F
+P 10100 4600
+F 0 "FID2" H 10185 4647 50  0000 L CNN
+F 1 "Fiducial" H 10185 4554 50  0000 L CNN
+F 2 "Fiducial:Fiducial_1.5mm_Mask4.5mm" H 10100 4600 50  0001 C CNN
+F 3 "~" H 10100 4600 50  0001 C CNN
+	1    10100 4600
+	1    0    0    -1
+$EndComp
+$Comp
+L Mechanical:Fiducial FID3
+U 1 1 607C95B1
+P 10100 4850
+F 0 "FID3" H 10185 4897 50  0000 L CNN
+F 1 "Fiducial" H 10185 4804 50  0000 L CNN
+F 2 "Fiducial:Fiducial_1.5mm_Mask4.5mm" H 10100 4850 50  0001 C CNN
+F 3 "~" H 10100 4850 50  0001 C CNN
+	1    10100 4850
+	1    0    0    -1
+$EndComp
 $EndSCHEMATC
